File: 04. Electronics/Crab Board v3/Crab_v3.sch (EAGLE design)
At the start: 29 parts, among them J1 JACK-2.1MM

Commit message: 1606
Connections:
- new net N$6: MICRO.PD0(RXD/PCINT16), PADS_2.1
Changed lines of the file:
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@@
+</segment>
+</net>
+<net name="N$6" class="0">
+<segment>
+<pinref part="MICRO" gate="1" pin="PD0(RXD/PCINT16)"/>
+<wire x1="71.12" y1="55.88" x2="165.1" y2="55.88" width="0.1524" layer="91"/>
+<wire x1="165.1" y1="55.88" x2="165.1" y2="38.1" width="0.1524" layer="91"/>
+<pinref part="PADS_2" gate="A" pin="1"/>
+<wire x1="165.1" y1="38.1" x2="175.26" y2="38.1" width="0.1524" layer="91"/>
 </segment>
 </net>
