File: 04. Electronics/Crab Board v3/Crab_v3.brd (EAGLE design)
At the start: 63.9 x 71.5 mm, 29 parts, among them J1 JACK-2.1MM

Commit message: 1606
Connections:
- new net N$6: MICRO.30, PADS_2.1
Routing:
- net N$6: track 0.00 -> 15.7 mm
Other:
- board size 63.9 x 71.5 mm -> 59.3 x 67.3 mm
Changed lines of the file:
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@@
 <layer number="16" name="Bottom" color="1" fill="1" visible="no" active="yes"/>
 <layer number="17" name="Pads" color="2" fill="1" visible="yes" active="yes"/>
-<layer number="18" name="Vias" color="2" fill="1" visible="no" active="yes"/>
+<layer number="18" name="Vias" color="2" fill="1" visible="yes" active="yes"/>
 <layer number="19" name="Unrouted" color="6" fill="1" visible="no" active="yes"/>
 <layer number="20" name="Dimension" color="15" fill="1" visible="yes" active="yes"/>
@@
 <board>
 <plain>
-<wire x1="12.827" y1="42.799" x2="76.708" y2="42.799" width="0.3048" layer="20"/>
-<wire x1="76.708" y1="42.799" x2="76.708" y2="-28.702" width="0.3048" layer="20"/>
-<wire x1="76.708" y1="-28.702" x2="12.827" y2="-28.702" width="0.3048" layer="20"/>
-<wire x1="12.827" y1="-28.702" x2="12.827" y2="42.799" width="0.3048" layer="20"/>
+<wire x1="15.367" y1="42.164" x2="74.549" y2="42.164" width="0.3048" layer="20"/>
+<wire x1="74.549" y1="42.164" x2="74.676" y2="-25.146" width="0.3048" layer="20"/>
+<wire x1="74.676" y1="-25.146" x2="15.621" y2="-25.019" width="0.3048" layer="20"/>
+<wire x1="15.621" y1="-25.019" x2="15.367" y2="42.164" width="0.3048" layer="20"/>
 </plain>
 <attributes>
@@
 <wire x1="61.432859375" y1="-23.41718125" x2="58.928" y2="-19.07863125" width="0.001" layer="1"/>
 </signal>
+<signal name="N$6">
+<contactref element="MICRO" pad="30"/>
+<contactref element="PADS_2" pad="1"/>
+<wire x1="45.79" y1="24.4856" x2="45.79" y2="32.131" width="0.3048" layer="1"/>
+<wire x1="45.79" y1="32.131" x2="41.021" y2="32.131" width="0.3048" layer="1"/>
+<wire x1="41.021" y1="32.131" x2="41.021" y2="35.433" width="0.3048" layer="1"/>
+</signal>
+<signal name="N$7">
+<via x="18.161" y="37.719" extent="1-16" drill="1.2" shape="octagon"/>
+</signal>
+<signal name="N$8">
+<via x="71.882" y="38.862" extent="1-16" drill="1.2" shape="octagon"/>
+</signal>
+<signal name="N$10">
+<via x="71.882" y="-22.098" extent="1-16" drill="1.2" shape="octagon"/>
+</signal>
+<signal name="N$11">
+<via x="36.195" y="-22.098" extent="1-16" drill="1.2" shape="octagon"/>
+</signal>
 </signals>

Commit message: 1706
Routing:
- net VCC: track 193.2 -> 183.6 mm
- net N$13: track 0.00 -> 5.08 mm
- net N$15: track 0.00 -> 4.50 mm
- net N$14: track 0.00 -> 4.50 mm
- net N$12: track 0.00 -> 3.81 mm
- net GND: track 228.4 -> 224.7 mm
- net N$22: track 19.0 -> 17.2 mm
- net N$11: track 0.00 -> 1.27 mm, vias 1 -> 0
- net P3: track 125.7 -> 126.5 mm
- net N$28: track 70.9 -> 71.7 mm
